Commit message: add: 夹爪优化

File: aubo/aubo_description/urdf/jiazhua.urdf (robot description, URDF)
Before this commit: robot jiazhua, 4 links, 3 joints
Joints:
- joint joint1: axis (none) -> 0 1 0; limit (none) -> lower=0.0 upper=0.55 effort=20.0 velocity=1.0; type fixed -> revolute
- joint joint2: axis (none) -> 0 1 0; limit (none) -> lower=0.0 upper=0.55 effort=20.0 velocity=1.0; type fixed -> revolute

Commit message: fix: 末端link平移

File: aubo/aubo_description/urdf/jiazhua.urdf (robot description, URDF)
Before this commit: robot jiazhua, 4 links, 3 joints
Links:
- added link tcp_link
Joints:
- added joint tcp_joint: type fixed, parent gripper_link, child tcp_link, origin xyz=0 0 0.025 rpy=0 0 0
