Commit message: add: mobile aubo

File: aubo/aubo_description/urdf/arm.xacro (robot description, xacro)
@@ -1,4 +1,8 @@
 <?xml version="1.0"?>
 <robot name="aubo_i5" xmlns:xacro="http://ros.org/wiki/xacro">
+ <!-- Keep the original stand-alone behaviour by default.  Composite robots can
+      disable the world joint and place ros_control in another namespace. -->
+    <xacro:arg name="standalone" default="true"/>
+    <xacro:arg name="robot_namespace" default="/aubo_i5"/>
  <!-- Defining the colors used in this robot -->
     <material name="Black">
@@ -298,10 +302,12 @@
 -->
  <!-- /////////////////////////////////   world   ////////////////////////////////////// -->
-  <link name="world" />
-  <joint name="world_joint" type="fixed">
-    <parent link="world" />
-    <child link ="base_link" />
-    <origin xyz="0.0 0.0 0.0" rpy="0.0 0.0 0.0" />
-  </joint>
+  <xacro:if value="$(arg standalone)">
+    <link name="world" />
+    <joint name="world_joint" type="fixed">
+      <parent link="world" />
+      <child link ="base_link" />
+      <origin xyz="0.0 0.0 0.0" rpy="0.0 0.0 0.0" />
+    </joint>
+  </xacro:if>
  <!-- /////////////////////////////////   jawasm1   //////////////////////////////////////
   <xacro:robotiq_85_gripper prefix="" parent="tool" >
@@ -336,5 +342,5 @@
   <gazebo>
       <plugin name="gazebo_ros_control" filename="libgazebo_ros_control.so">
-          <robotNamespace>/aubo_i5</robotNamespace>
+          <robotNamespace>$(arg robot_namespace)</robotNamespace>
 	        <robotSimType>gazebo_ros_control/DefaultRobotHWSim</robotSimType>
           <legacyModeNS>true</legacyModeNS>

Commit message: fix: 修改抓取场景 增加shoulder_joint限位

File: aubo/aubo_description/urdf/arm.xacro (robot description, xacro)
@@ -140,5 +140,7 @@
     <child link="shoulder_Link" />
     <axis xyz="0 0 1" />
-    <limit lower="-3.04" upper="3.04" effort="300" velocity="100" />
+    <!-- Keep the shoulder away from the table-side rear sweep:
+         -90 deg + 10 deg <= q <= 90 deg - 10 deg. -->
+    <limit lower="-1.3962634" upper="1.3962634" effort="300" velocity="100" />
   </joint>
   <!--/////////////////////////////// UPPERARM_LINK ////////////////////////////////////-->

Commit message: fix: Gazebo 接触参数

File: aubo/aubo_description/urdf/arm.xacro (robot description, xacro)
@@ -140,7 +140,6 @@
     <child link="shoulder_Link" />
     <axis xyz="0 0 1" />
-    <!-- Keep the shoulder away from the table-side rear sweep:
-         -90 deg + 10 deg <= q <= 90 deg - 10 deg. -->
-    <limit lower="-1.3962634" upper="1.3962634" effort="300" velocity="100" />
+    <!-- Limit the table-side shoulder sweep to -50 deg ... +50 deg. -->
+    <limit lower="-0.8726646" upper="0.8726646" effort="300" velocity="100" />
   </joint>
   <!--/////////////////////////////// UPPERARM_LINK ////////////////////////////////////-->

Commit message: fix: 关节限位调整，修改目标参数

File: aubo/aubo_description/urdf/arm.xacro (robot description, xacro)
@@ -140,6 +140,5 @@
     <child link="shoulder_Link" />
     <axis xyz="0 0 1" />
-    <!-- Limit the table-side shoulder sweep to -50 deg ... +50 deg. -->
-    <limit lower="-0.8726646" upper="0.8726646" effort="300" velocity="100" />
+    <limit lower="-3.04" upper="3.04" effort="300" velocity="100" />
   </joint>
   <!--/////////////////////////////// UPPERARM_LINK ////////////////////////////////////-->
@@ -170,5 +169,6 @@
     <child link="upperArm_Link" />
     <axis xyz="0 0 1" />
-    <limit lower="-3.04" upper="3.04" effort="300" velocity="100" />
+    <!-- Restrict the second actuated joint to -60 deg ... +60 deg. -->
+    <limit lower="-1.0471976" upper="1.0471976" effort="300" velocity="100" />
   </joint>
   <!--/////////////////////////////// FOREARM_LINK ////////////////////////////////////-->

File: aubo/aubo_description/urdf/jiazhua.urdf (robot description, URDF)
Before this commit: robot jiazhua, 5 links, 4 joints
Joints:
- joint tcp_joint: origin xyz=0 0 0.025 rpy=0 0 0 -> xyz=0 0 0 rpy=0 0 0
