Commit message: add: object dector

File: aubo/aubo_description/urdf/hand_camera.xacro (robot description, xacro)
@@ -1,5 +1,5 @@
 <?xml version="1.0"?>
 <robot name="aubo_hand_camera" xmlns:xacro="http://www.ros.org/wiki/xacro">
-  <!-- Eye-in-hand RGB camera adapted from the mobile manipulator model.
+  <!-- Eye-in-hand RGB-D camera with RealSense-compatible ROS topic names.
        Camera optical conventions: +Z forward, +X right, +Y down. -->
   <xacro:macro name="aubo_hand_camera" params="parent_link">
@@ -61,4 +61,36 @@
       <origin xyz="0.03 0 0" rpy="-1.57079632679 0 -1.57079632679"/>
     </joint>
+    <!-- Standard RealSense frame aliases.  Keep the old hand_camera frame for
+         compatibility with the sorting package while new code uses these. -->
+    <link name="camera_link"/>
+    <joint name="camera_link_joint" type="fixed">
+      <parent link="hand_camera_link"/>
+      <child link="camera_link"/>
+      <origin xyz="0 0 0" rpy="0 0 0"/>
+    </joint>
+    <link name="camera_color_frame"/>
+    <joint name="camera_color_joint" type="fixed">
+      <parent link="camera_link"/>
+      <child link="camera_color_frame"/>
+      <origin xyz="0.03 0 0" rpy="0 0 0"/>
+    </joint>
+    <link name="camera_color_optical_frame"/>
+    <joint name="camera_color_optical_joint" type="fixed">
+      <parent link="camera_color_frame"/>
+      <child link="camera_color_optical_frame"/>
+      <origin xyz="0 0 0" rpy="-1.57079632679 0 -1.57079632679"/>
+    </joint>
+    <link name="camera_depth_frame"/>
+    <joint name="camera_depth_joint" type="fixed">
+      <parent link="camera_link"/>
+      <child link="camera_depth_frame"/>
+      <origin xyz="0.03 0 0" rpy="0 0 0"/>
+    </joint>
+    <link name="camera_depth_optical_frame"/>
+    <joint name="camera_depth_optical_joint" type="fixed">
+      <parent link="camera_depth_frame"/>
+      <child link="camera_depth_optical_frame"/>
+      <origin xyz="0 0 0" rpy="-1.57079632679 0 -1.57079632679"/>
+    </joint>
     <gazebo reference="hand_camera_mount_link">
       <material>Gazebo/Black</material>
@@ -66,10 +98,10 @@
     <gazebo reference="hand_camera_link">
       <material>Gazebo/Grey</material>
-      <sensor type="camera" name="hand_camera">
+      <sensor type="depth" name="hand_realsense">
         <pose>0.03 0 0 0 0 0</pose>
         <always_on>true</always_on>
         <visualize>false</visualize>
         <update_rate>20</update_rate>
-        <camera name="hand_camera_sensor">
+        <camera name="hand_realsense_sensor">
           <horizontal_fov>1.047</horizontal_fov>
           <image>
@@ -80,9 +112,25 @@
           <clip><near>0.05</near><far>20.0</far></clip>
         </camera>
-        <plugin name="hand_gazebo_ros_camera" filename="libgazebo_ros_camera.so">
-          <cameraName>hand_camera</cameraName>
-          <imageTopicName>image_raw</imageTopicName>
-          <cameraInfoTopicName>camera_info</cameraInfoTopicName>
-          <frameName>hand_camera_optical_frame</frameName>
+        <plugin name="hand_gazebo_realsense" filename="libgazebo_ros_openni_kinect.so">
+          <robotNamespace>/</robotNamespace>
+          <cameraName>camera</cameraName>
+          <alwaysOn>true</alwaysOn>
+          <updateRate>20.0</updateRate>
+          <imageTopicName>color/image_raw</imageTopicName>
+          <cameraInfoTopicName>color/camera_info</cameraInfoTopicName>
+          <!-- The simulated depth sensor shares the color optical centre, so
+               its depth image is already aligned to the color image. -->
+          <depthImageTopicName>aligned_depth_to_color/image_raw</depthImageTopicName>
+          <depthImageCameraInfoTopicName>aligned_depth_to_color/camera_info</depthImageCameraInfoTopicName>
+          <pointCloudTopicName>depth/color/points</pointCloudTopicName>
+          <frameName>camera_color_optical_frame</frameName>
+          <baseline>0.05</baseline>
+          <pointCloudCutoff>0.08</pointCloudCutoff>
+          <pointCloudCutoffMax>4.0</pointCloudCutoffMax>
+          <distortion_k1>0.0</distortion_k1>
+          <distortion_k2>0.0</distortion_k2>
+          <distortion_k3>0.0</distortion_k3>
+          <distortion_t1>0.0</distortion_t1>
+          <distortion_t2>0.0</distortion_t2>
         </plugin>
       </sensor>

Commit message: fix: 相机位置调整

File: aubo/aubo_description/urdf/hand_camera.xacro (robot description, xacro)
@@ -6,23 +6,35 @@
     <link name="hand_camera_mount_link">
       <visual>
-        <origin xyz="0 -0.035 0.055" rpy="0 0 0"/>
-        <geometry><box size="0.024 0.070 0.012"/></geometry>
+        <!-- 安装底板：固定在夹爪基座中心。 -->
+        <origin xyz="0 0 0.020" rpy="0 0 0"/>
+        <geometry><box size="0.050 0.050 0.012"/></geometry>
         <material name="hand_camera_black"><color rgba="0.025 0.03 0.04 1"/></material>
       </visual>
       <visual>
-        <origin xyz="0.020 -0.070 0.055" rpy="0 0 0"/>
-        <geometry><box size="0.040 0.024 0.012"/></geometry>
+        <!-- 竖向支柱：连接安装底板与相机横梁。 -->
+        <origin xyz="0 0 0.0375" rpy="0 0 0"/>
+        <geometry><box size="0.024 0.024 0.035"/></geometry>
+        <material name="hand_camera_black"/>
+      </visual>
+      <visual>
+        <!-- 相机横梁：沿 X 方向延伸 60 mm，Y 方向保持居中。 -->
+        <origin xyz="0.030 0 0.055" rpy="0 0 0"/>
+        <geometry><box size="0.060 0.024 0.012"/></geometry>
         <material name="hand_camera_black"/>
       </visual>
       <collision>
-        <origin xyz="0 -0.035 0.055" rpy="0 0 0"/>
-        <geometry><box size="0.024 0.070 0.012"/></geometry>
+        <origin xyz="0 0 0.020" rpy="0 0 0"/>
+        <geometry><box size="0.050 0.050 0.012"/></geometry>
       </collision>
       <collision>
-        <origin xyz="0.020 -0.070 0.055" rpy="0 0 0"/>
-        <geometry><box size="0.040 0.024 0.012"/></geometry>
+        <origin xyz="0 0 0.0375" rpy="0 0 0"/>
+        <geometry><box size="0.024 0.024 0.035"/></geometry>
+      </collision>
+      <collision>
+        <origin xyz="0.030 0 0.055" rpy="0 0 0"/>
+        <geometry><box size="0.060 0.024 0.012"/></geometry>
       </collision>
       <inertial>
-        <origin xyz="0.010 -0.050 0.055" rpy="0 0 0"/>
+        <origin xyz="0.025 0 0.045" rpy="0 0 0"/>
         <mass value="0.12"/>
         <inertia ixx="0.000066" ixy="0" ixz="0"
@@ -52,6 +64,7 @@
       <parent link="hand_camera_mount_link"/>
       <child link="hand_camera_link"/>
-      <!-- Gazebo camera looks along local +X; align it with the gripper approach axis. -->
-      <origin xyz="0.040 -0.070 0.055" rpy="0 -1.57079632679 0"/>
+      <!-- 相机相对夹爪沿 X 方向偏移 60 mm，Y 方向无侧向偏移。
+           相机局部 +X 方向旋转后指向夹爪的 +Z 工作方向。 -->
+      <origin xyz="0.060 0 0.055" rpy="0 -1.57079632679 0"/>
     </joint>
     <link name="hand_camera_optical_frame"/>

File: aubo_mobile_robot/aubo_mobile_robot/urdf/aubo_mobile_robot.xacro (robot description, xacro)
@@ -265,37 +265,52 @@
   <xacro:planar_lidar name="front" x="0.27" yaw="0" topic="front/scan"/>
   <xacro:planar_lidar name="rear" x="-0.27" yaw="${pi}" topic="rear/scan"/>
-  <!-- Camera mounted beside the hand; optical frame follows REP-103. It can
-       be omitted for external-camera tasks to avoid duplicate image streams. -->
+  <!-- 眼在手相机安装在夹爪的 Y 向中心平面上，光学坐标系遵循 REP-103。
+       使用外部相机时可关闭该模型，避免产生重复图像话题。 -->
   <xacro:if value="$(arg enable_hand_camera)">
   <link name="hand_camera_mount_link">
-    <!-- Two bars form an L bracket from the gripper body to the side camera. -->
-    <visual>
-      <origin xyz="0 -0.035 0.055" rpy="0 0 0"/>
-      <geometry>
-        <box size="0.024 0.070 0.012"/>
+    <!-- 安装底板：固定在夹爪基座中心。 -->
+    <visual>
+      <origin xyz="0 0 0.020" rpy="0 0 0"/>
+      <geometry>
+        <box size="0.050 0.050 0.012"/>
       </geometry>
       <material name="mobile_dark"/>
     </visual>
     <visual>
-      <origin xyz="0.020 -0.070 0.055" rpy="0 0 0"/>
-      <geometry>
-        <box size="0.040 0.024 0.012"/>
+      <!-- 竖向支柱：连接安装底板与相机横梁。 -->
+      <origin xyz="0 0 0.0375" rpy="0 0 0"/>
+      <geometry>
+        <box size="0.024 0.024 0.035"/>
       </geometry>
       <material name="mobile_dark"/>
     </visual>
-    <collision>
-      <origin xyz="0 -0.035 0.055" rpy="0 0 0"/>
-      <geometry>
-        <box size="0.024 0.070 0.012"/>
-      </geometry>
-    </collision>
-    <collision>
-      <origin xyz="0.020 -0.070 0.055" rpy="0 0 0"/>
-      <geometry>
-        <box size="0.040 0.024 0.012"/>
+    <visual>
+      <!-- 相机横梁：沿 X 方向延伸 60 mm，Y 方向保持居中。 -->
+      <origin xyz="0.030 0 0.055" rpy="0 0 0"/>
+      <geometry>
+        <box size="0.060 0.024 0.012"/>
+      </geometry>
+      <material name="mobile_dark"/>
+    </visual>
+    <collision>
+      <origin xyz="0 0 0.020" rpy="0 0 0"/>
+      <geometry>
+        <box size="0.050 0.050 0.012"/>
+      </geometry>
+    </collision>
+    <collision>
+      <origin xyz="0 0 0.0375" rpy="0 0 0"/>
+      <geometry>
+        <box size="0.024 0.024 0.035"/>
+      </geometry>
+    </collision>
+    <collision>
+      <origin xyz="0.030 0 0.055" rpy="0 0 0"/>
+      <geometry>
+        <box size="0.060 0.024 0.012"/>
       </geometry>
     </collision>
     <inertial>
-      <origin xyz="0.010 -0.050 0.055" rpy="0 0 0"/>
+      <origin xyz="0.025 0 0.045" rpy="0 0 0"/>
       <mass value="0.12"/>
       <inertia ixx="0.000066" ixy="0" ixz="0" iyy="0.000018" iyz="0" izz="0.000080"/>
@@ -327,7 +342,7 @@
     <parent link="hand_camera_mount_link"/>
     <child link="hand_camera_link"/>
-    <!-- Gazebo cameras look along local +X. Rotate +X onto the gripper's +Z
-         approach axis so a downward grasp pose also looks at the table. -->
-    <origin xyz="0.040 -0.070 0.055" rpy="0 ${-pi / 2.0} 0"/>
+    <!-- 相机相对夹爪沿 X 方向偏移 60 mm，Y 方向无侧向偏移。
+         相机局部 +X 方向旋转后指向夹爪的 +Z 工作方向。 -->
+    <origin xyz="0.060 0 0.055" rpy="0 ${-pi / 2.0} 0"/>
   </joint>
   <link name="hand_camera_optical_frame"/>
