Commit message: add: aubo模型加上眼在手上 相机

File: aubo/aubo_description/urdf/aubo_i5_with_camera.xacro (robot description, xacro)
@@ -1,23 +1,13 @@
 <?xml version="1.0"?>
 <robot name="aubo_i5" xmlns:xacro="http://www.ros.org/wiki/xacro">
-  <xacro:property name="M_PI" value="3.14159"/>
-  <xacro:property name="PI" value="3.14159"/>
-   <!--camera position-->
-   <xacro:property name="camera_offset_x" value="0" />
-   <xacro:property name="camera_offset_y" value="-0.75" />
-   <xacro:property name="camera_offset_z" value="1" />
-   <xacro:include filename="$(find aubo_description)/urdf/camera.xacro"/>
-  <xacro:include filename="$(find aubo_description)/urdf/jiazhua.urdf" />
-  <xacro:include filename="$(find aubo_description)/urdf/arm.xacro" />
-    <joint name="ee_link_joint" type="fixed">
-        <origin xyz="0 0 0" rpy="0 0 0 " />
-        <parent link="wrist3_Link" />
-        <child  link="gripper_base_link" />
-    </joint>
- <!--Camera -->
-    <joint name="camera_joint" type="fixed">
-        <origin xyz="${camera_offset_x} ${camera_offset_y} ${camera_offset_z}" rpy="${-M_PI/2} ${M_PI/2} ${-M_PI/2}" />
-        <parent link="base_link" />
-        <child  link="camera_link" />
-    </joint>
+  <xacro:property name="M_PI" value="3.141592653589793"/>
+  <xacro:include filename="$(find aubo_description)/urdf/jiazhua.urdf"/>
+  <xacro:include filename="$(find aubo_description)/urdf/arm.xacro"/>
+  <xacro:include filename="$(find aubo_description)/urdf/hand_camera.xacro"/>
+  <joint name="ee_link_joint" type="fixed">
+    <parent link="wrist3_Link"/>
+    <child link="gripper_base_link"/>
+    <origin xyz="0 0 0" rpy="0 0 0"/>
+  </joint>
+  <xacro:aubo_hand_camera parent_link="gripper_base_link"/>
 </robot>

Commit message: fix: 分拣修正

File: aubo/aubo_description/urdf/aubo_i5_with_camera.xacro (robot description, xacro)
@@ -2,4 +2,9 @@
 <robot name="aubo_i5" xmlns:xacro="http://www.ros.org/wiki/xacro">
   <xacro:property name="M_PI" value="3.141592653589793"/>
+  <xacro:arg name="camera_horizontal_fov" default="1.3962634016"/>
+  <xacro:arg name="camera_lateral_offset" default="0.060"/>
+  <xacro:arg name="camera_mount_z_shift" default="0.0"/>
+  <xacro:arg name="camera_clip_near" default="0.05"/>
+  <xacro:arg name="camera_pointcloud_cutoff" default="0.08"/>
   <xacro:include filename="$(find aubo_description)/urdf/jiazhua.urdf"/>
   <xacro:include filename="$(find aubo_description)/urdf/arm.xacro"/>
@@ -10,4 +15,9 @@
     <origin xyz="0 0 0" rpy="0 0 0"/>
   </joint>
-  <xacro:aubo_hand_camera parent_link="gripper_base_link"/>
+  <xacro:aubo_hand_camera parent_link="gripper_base_link"
+      horizontal_fov="$(arg camera_horizontal_fov)"
+      lateral_offset="$(arg camera_lateral_offset)"
+      mount_z_shift="$(arg camera_mount_z_shift)"
+      clip_near="$(arg camera_clip_near)"
+      pointcloud_cutoff="$(arg camera_pointcloud_cutoff)"/>
 </robot>

File: aubo/aubo_description/urdf/hand_camera.xacro (robot description, xacro)
@@ -3,9 +3,9 @@
   <!-- Eye-in-hand RGB-D camera with RealSense-compatible ROS topic names.
        Camera optical conventions: +Z forward, +X right, +Y down. -->
-  <xacro:macro name="aubo_hand_camera" params="parent_link">
+  <xacro:macro name="aubo_hand_camera" params="parent_link lateral_offset:=0.060 mount_z_shift:=0.0 horizontal_fov:=1.3962634016 clip_near:=0.05 pointcloud_cutoff:=0.08">
     <link name="hand_camera_mount_link">
       <visual>
         <!-- 安装底板：固定在夹爪基座中心。 -->
-        <origin xyz="0 0 0.020" rpy="0 0 0"/>
+        <origin xyz="0 0 ${0.020 + mount_z_shift}" rpy="0 0 0"/>
         <geometry><box size="0.050 0.050 0.012"/></geometry>
         <material name="hand_camera_black"><color rgba="0.025 0.03 0.04 1"/></material>
@@ -13,5 +13,5 @@
       <visual>
         <!-- 竖向支柱：连接安装底板与相机横梁。 -->
-        <origin xyz="0 0 0.0375" rpy="0 0 0"/>
+        <origin xyz="0 0 ${0.0375 + mount_z_shift}" rpy="0 0 0"/>
         <geometry><box size="0.024 0.024 0.035"/></geometry>
         <material name="hand_camera_black"/>
@@ -19,22 +19,22 @@
       <visual>
         <!-- 相机横梁：沿 X 方向延伸 60 mm，Y 方向保持居中。 -->
-        <origin xyz="0.030 0 0.055" rpy="0 0 0"/>
-        <geometry><box size="0.060 0.024 0.012"/></geometry>
+        <origin xyz="${lateral_offset / 2} 0 ${0.055 + mount_z_shift}" rpy="0 0 0"/>
+        <geometry><box size="${lateral_offset} 0.024 0.012"/></geometry>
         <material name="hand_camera_black"/>
       </visual>
       <collision>
-        <origin xyz="0 0 0.020" rpy="0 0 0"/>
+        <origin xyz="0 0 ${0.020 + mount_z_shift}" rpy="0 0 0"/>
         <geometry><box size="0.050 0.050 0.012"/></geometry>
       </collision>
       <collision>
-        <origin xyz="0 0 0.0375" rpy="0 0 0"/>
+        <origin xyz="0 0 ${0.0375 + mount_z_shift}" rpy="0 0 0"/>
         <geometry><box size="0.024 0.024 0.035"/></geometry>
       </collision>
       <collision>
-        <origin xyz="0.030 0 0.055" rpy="0 0 0"/>
-        <geometry><box size="0.060 0.024 0.012"/></geometry>
+        <origin xyz="${lateral_offset / 2} 0 ${0.055 + mount_z_shift}" rpy="0 0 0"/>
+        <geometry><box size="${lateral_offset} 0.024 0.012"/></geometry>
       </collision>
       <inertial>
-        <origin xyz="0.025 0 0.045" rpy="0 0 0"/>
+        <origin xyz="${0.025 + 0.5 * (lateral_offset - 0.060)} 0 ${0.045 + mount_z_shift}" rpy="0 0 0"/>
         <mass value="0.12"/>
         <inertia ixx="0.000066" ixy="0" ixz="0"
@@ -66,5 +66,5 @@
       <!-- 相机相对夹爪沿 X 方向偏移 60 mm，Y 方向无侧向偏移。
            相机局部 +X 方向旋转后指向夹爪的 +Z 工作方向。 -->
-      <origin xyz="0.060 0 0.055" rpy="0 -1.57079632679 0"/>
+      <origin xyz="${lateral_offset} 0 ${0.055 + mount_z_shift}" rpy="0 -1.57079632679 0"/>
     </joint>
     <link name="hand_camera_optical_frame"/>
@@ -119,5 +119,5 @@
           <!-- 80 deg horizontal FOV: wide enough to acquire targets during
                eye-in-hand search without excessive edge perspective. -->
-          <horizontal_fov>1.3962634016</horizontal_fov>
+          <horizontal_fov>${horizontal_fov}</horizontal_fov>
           <image>
             <width>1280</width>
@@ -125,5 +125,5 @@
             <format>R8G8B8</format>
           </image>
-          <clip><near>0.05</near><far>20.0</far></clip>
+          <clip><near>${clip_near}</near><far>20.0</far></clip>
         </camera>
         <plugin name="hand_gazebo_realsense" filename="libgazebo_ros_openni_kinect.so">
@@ -141,5 +141,5 @@
           <frameName>camera_color_optical_frame</frameName>
           <baseline>0.05</baseline>
-          <pointCloudCutoff>0.08</pointCloudCutoff>
+          <pointCloudCutoff>${pointcloud_cutoff}</pointCloudCutoff>
           <pointCloudCutoffMax>4.0</pointCloudCutoffMax>
           <distortion_k1>0.0</distortion_k1>
