Commit message: 修改模型问题-不平衡移动问题，还存在问题 移动过程中雷达偏移

File: simple_diff_robot_gazebo/urdf/simple_diff_robot.xacro (robot description, xacro)
@@ -66,5 +66,5 @@
       <child link="${side}_wheel_link"/>
       <origin xyz="0 ${y} 0" rpy="${pi / 2.0} 0 0"/>
-      <axis xyz="0 0 1"/>
+      <axis xyz="0 0 -1"/>
       <dynamics damping="0.05" friction="0.0"/>
     </joint>
@@ -93,4 +93,24 @@
     <origin xyz="${caster_x} 0 ${caster_radius - wheel_radius}"/>
   </joint>
+  <link name="caster_link2">
+    <visual>
+      <geometry><sphere radius="${caster_radius}"/></geometry>
+      <material name="silver"/>
+    </visual>
+    <collision>
+      <geometry><sphere radius="${caster_radius}"/></geometry>
+    </collision>
+    <inertial>
+      <mass value="${caster_mass}"/>
+      <inertia ixx="${0.4 * caster_mass * caster_radius * caster_radius}" ixy="0" ixz="0"
+               iyy="${0.4 * caster_mass * caster_radius * caster_radius}" iyz="0"
+               izz="${0.4 * caster_mass * caster_radius * caster_radius}"/>
+    </inertial>
+  </link>
+  <joint name="caster_joint2" type="fixed">
+    <parent link="base_link"/>
+    <child link="caster_link2"/>
+    <origin xyz="${-caster_x} 0 ${caster_radius - wheel_radius}"/>
+  </joint>
   <!-- 2D lidar, mounted above the chassis. -->
   <link name="laser_link">
@@ -111,5 +131,5 @@
   <joint name="camera_joint" type="fixed">
     <parent link="base_link"/><child link="camera_link"/>
-    <origin xyz="${base_length / 2.0 - 0.025} 0 ${base_height + 0.06}"/>
+    <origin xyz="${base_length / 2.0 - 0.025} 0 ${base_height}"/>
   </joint>
   <link name="camera_optical_frame"/>
@@ -128,4 +148,9 @@
     <material>Gazebo/Grey</material>
     <mu1>0.001</mu1><mu2>0.001</mu2>
+  </gazebo>
+  <gazebo reference="caster_link2">
+    <material>Gazebo/Grey</material>
+    <mu1>0.001</mu1>
+    <mu2>0.001</mu2>
   </gazebo>
   <gazebo reference="laser_link">

Commit message: fix: 修改里程计偏移问题

File: simple_diff_robot_gazebo/urdf/simple_diff_robot.xacro (robot description, xacro)
@@ -140,8 +140,8 @@
   <gazebo reference="base_link"><material>Gazebo/Blue</material></gazebo>
   <gazebo reference="left_wheel_link">
-    <material>Gazebo/Black</material><mu1>1.0</mu1><mu2>1.0</mu2>
+    <material>Gazebo/Black</material><mu1>2.0</mu1><mu2>2.0</mu2>
   </gazebo>
   <gazebo reference="right_wheel_link">
-    <material>Gazebo/Black</material><mu1>1.0</mu1><mu2>1.0</mu2>
+    <material>Gazebo/Black</material><mu1>2.0</mu1><mu2>2.0</mu2>
   </gazebo>
   <gazebo reference="caster_link">
@@ -196,6 +196,8 @@
       <odometryFrame>odom</odometryFrame>
       <robotBaseFrame>base_footprint</robotBaseFrame>
-      <!-- Encoder odometry is more realistic for learning SLAM than Gazebo world ground truth. -->
-      <odometrySource>encoder</odometrySource>
+      <!-- Demo/navigation mode: world ground-truth odometry keeps the local costmap and
+           laser perfectly aligned (no encoder drift). For learning SLAM on realistic
+           odometry, switch back to: <odometrySource>encoder</odometrySource> -->
+      <odometrySource>world</odometrySource>
       <publishOdomTF>true</publishOdomTF>
       <publishWheelTF>false</publishWheelTF>

Commit message: fix：dwa局部规划器问题

File: simple_diff_robot_gazebo/urdf/simple_diff_robot.xacro (robot description, xacro)
@@ -140,8 +140,8 @@
   <gazebo reference="base_link"><material>Gazebo/Blue</material></gazebo>
   <gazebo reference="left_wheel_link">
-    <material>Gazebo/Black</material><mu1>2.0</mu1><mu2>2.0</mu2>
+    <material>Gazebo/Black</material><mu1>1.0</mu1><mu2>1.0</mu2>
   </gazebo>
   <gazebo reference="right_wheel_link">
-    <material>Gazebo/Black</material><mu1>2.0</mu1><mu2>2.0</mu2>
+    <material>Gazebo/Black</material><mu1>1.0</mu1><mu2>1.0</mu2>
   </gazebo>
   <gazebo reference="caster_link">
@@ -197,6 +197,10 @@
       <robotBaseFrame>base_footprint</robotBaseFrame>
       <!-- Demo/navigation mode: world ground-truth odometry keeps the local costmap and
-           laser perfectly aligned (no encoder drift). For learning SLAM on realistic
-           odometry, switch back to: <odometrySource>encoder</odometrySource> -->
+           laser perfectly aligned (no encoder drift). NOTE: do NOT combine this with
+           high wheel friction -- with mu 2.0 the robot physically wedges against
+           obstacles and, because world odom no longer masks the stall with drift,
+           DWA reports "failed to produce path" and recovery cannot free it.
+           For learning SLAM on realistic odometry, switch back to:
+           <odometrySource>encoder</odometrySource> -->
       <odometrySource>world</odometrySource>
       <publishOdomTF>true</publishOdomTF>

Commit message: fix: 差速小车 simple follower

File: simple_diff_robot_gazebo/urdf/simple_diff_robot.xacro (robot description, xacro)
@@ -1,4 +1,5 @@
 <?xml version="1.0"?>
 <robot name="simple_diff_robot" xmlns:xacro="http://www.ros.org/wiki/xacro">
+  <xacro:arg name="camera_pitch" default="0.0"/>
   <!-- All dimensions are in metres and kilograms. -->
   <xacro:property name="base_length" value="0.40"/>
@@ -131,5 +132,5 @@
   <joint name="camera_joint" type="fixed">
     <parent link="base_link"/><child link="camera_link"/>
-    <origin xyz="${base_length / 2.0 - 0.025} 0 ${base_height}"/>
+    <origin xyz="${base_length / 2.0 - 0.025} 0 ${base_height}" rpy="0 $(arg camera_pitch) 0"/>
   </joint>
   <link name="camera_optical_frame"/>
